Commit message: rotated forklift model to align with convention. x is forward

File: forklift_description/urdf/forklift.xacro (robot description, xacro)
@@ -4,9 +4,9 @@
   <!-- Constants for robot dimensions -->
   <xacro:property name="PI" value="3.1415926535897931"/>
-  <xacro:property name="body_mass" value="50" />
+  <xacro:property name="body_mass" value="1" />
   <xacro:property name="lift1_mass" value="10" />
   <xacro:property name="lift2_mass" value="10" />
   <xacro:property name="wheelF_mass" value="10" />
-  <xacro:property name="wheelB_mass" value="0.1" />
+  <xacro:property name="wheelB_mass" value="5" />
   <xacro:property name="wheelF_radius" value="0.33" />
   <xacro:property name="wheelF_width" value="0.01" />
@@ -26,18 +26,18 @@
   <xacro:macro name="cube_inertia" params="m w h d">
           <inertia
-            ixx="${m / 12.0 * (d*d + h*h)}" ixy="0.0" ixz="0.0"
-            iyy="${m / 12.0 * (w*w + h*h)}" iyz="0.0"
-            izz="${m / 12.0 * (w*w + d*d)}"/>
+            ixx="${m / 12.0 * (h*h + d*d)}" ixy="0.0" ixz="0.0"
+            iyy="${m / 12.0 * (d*d + w*w)}" iyz="0.0"
+            izz="${m / 12.0 * (h*h + w*w)}"/>
   </xacro:macro>
   <!-- Forklift -->
-  <link name="forklift_body">
+  <link name="base_link">
     <collision>
-      <origin xyz="0 0 ${height/2 + 0.2}" rpy="0 0 0"/>
+      <origin xyz="-1 0 ${height/2 + 0.2}" rpy="0 0 0"/>
       <geometry>
-	     <box size="${width} ${length} ${height}"/>
+	     <box size="${length} ${width} ${height}"/>
       </geometry>
     </collision>
     <visual>
-      <origin xyz="-0.00203 -0.06282 1.08726" rpy="0 0 0"/>
+      <origin xyz="-0.89856 0 1.08726" rpy="0 0 ${PI/2}"/> <!-- -0.00203 -0.06282 1.08726-->
       <geometry>
 	     <mesh filename="package://forklift_description/meshes/forklift_body.dae"/>
@@ -45,16 +45,9 @@
     </visual>
     <inertial>
-      <origin xyz="0.3 0 1" rpy="0 0 0"/>
+      <origin xyz="0 0 1" rpy="0 0 0"/>
       <mass value="${body_mass}"/>
-      <cube_inertia m="${body_mass}" w="1.3" h="2" d="2" />
+      <cube_inertia m="${lift1_mass}" w="1" h="1" d="1" />
     </inertial>
   </link>
-  <!-- caster Wheel -->
-  <joint name="caster_wheel_joint" type="continuous">
-    <parent link="forklift_body"/>
-    <child link="caster_wheel"/>
-    <origin xyz="0.0 0.76717 0.27997" rpy="0 ${PI/2} 0" />
-    <axis xyz="0 0 1" />
-  </joint>
   <!-- Import lift unit -->
   <xacro:include filename="$(find forklift_description)/urdf/forklift_lift.xacro" />

File: forklift_description/urdf/forklift_back_wheels.xacro (robot description, xacro)
@@ -20,8 +20,8 @@
   <!-- BR Wheel -->
   <joint name="wheelBR_joint" type="fixed">
-    <parent link="forklift_body"/>
+    <parent link="base_link"/>
     <child link="forklift_wheelBR"/>
-    <axis xyz="1 0 0"/>
-    <origin xyz="-0.49259 0.76717 0.27997" />
+    <axis xyz="0 1 0"/>
+    <origin xyz="-1.730949 -0.49259 0.27997" /> <!-- -0.49259 0.76717 0.27997 -->
   </joint>
   <link name="forklift_wheelBR">
@@ -35,5 +35,5 @@
     -->
     <visual>
-      <origin xyz="0 0 0" rpy="0 0 ${PI}"/>
+      <origin xyz="0 0 0" rpy="0 0 ${PI+PI/2}"/>
       <geometry>
        <mesh filename="package://forklift_description/meshes/forklift_wheel_back.dae"/>
@@ -41,5 +41,5 @@
     </visual>
     <inertial>
-      <origin xyz="0 0 0" rpy="0 ${PI/2} 0"/>
+      <origin xyz="0 0 0" rpy="0 0 0"/>
       <mass value="${wheelF_mass}"/>
       <cylinder_inertia  m="${wheelB_mass}" r="${wheelB_radius}" h="${wheelB_width}" />
@@ -65,8 +65,8 @@
   <!-- BL Wheel -->
   <joint name="wheelBL_joint" type="fixed">
-    <parent link="forklift_body"/>
+    <parent link="base_link"/>
     <child link="forklift_wheelBL"/>
-    <axis xyz="1 0 0"/>
-    <origin xyz="0.49259 0.76717 0.27997" />
+    <axis xyz="0 1 0"/>
+    <origin xyz="-1.730949 0.49259 0.27997" />
   </joint>
   <link name="forklift_wheelBL">
@@ -80,5 +80,5 @@
   -->
     <visual>
-      <origin xyz="0 0 0" rpy="0 0 0"/>
+      <origin xyz="0 0 0" rpy="0 0 ${PI/2}"/>
       <geometry>
        <mesh filename="package://forklift_description/meshes/forklift_wheel_back.dae"/>
@@ -86,9 +86,16 @@
     </visual>
     <inertial>
-      <origin xyz="0 0 0" rpy="0 ${PI/2} 0"/>
+      <origin xyz="0 0 0" rpy="0 0 0"/>
       <mass value="${wheelF_mass}"/>
       <cylinder_inertia  m="${wheelB_mass}" r="${wheelB_radius}" h="${wheelB_width}" />
     </inertial>
   </link>
+  <!-- caster Wheel -->
+  <joint name="caster_wheel_joint" type="continuous">
+    <parent link="base_link"/>
+    <child link="caster_wheel"/>
+    <origin xyz="-1.76717 0 0.27997" rpy="0 ${PI/2} 0" />
+    <axis xyz="0 0 1" />
+  </joint>
   <link name="caster_wheel">
     <collision>

File: forklift_description/urdf/forklift_front_wheels.xacro (robot description, xacro)
@@ -3,12 +3,12 @@
   <!-- FR Wheel -->
   <joint name="wheelFR_joint" type="continuous">
-    <parent link="forklift_body"/>
+    <parent link="base_link"/>
     <child link="forklift_wheelFR"/>
-    <axis xyz="1 0 0"/>
-    <origin xyz="-0.49389 -0.90059 0.34047"/>
+    <axis xyz="0 1 0"/>
+    <origin xyz="0 -0.49389 0.34047"/>
   </joint>
   <link name="forklift_wheelFR">
     <collision>
-      <origin xyz="0 0 0" rpy="0 ${PI/2} 0"/>
+      <origin xyz="0 0 0" rpy="${PI/2} 0 0"/>
       <geometry>
        <cylinder radius="${wheelF_radius}" length="${wheelF_width}" />
@@ -16,5 +16,5 @@
     </collision>
     <visual>
-      <origin xyz="0 0 0" rpy="0 0 ${PI}"/>
+      <origin xyz="0 0 0" rpy="0 0 ${PI+PI/2}"/>
       <geometry>
        <mesh filename="package://forklift_description/meshes/forklift_wheel_front.dae"/>
@@ -22,5 +22,5 @@
     </visual>
     <inertial>
-      <origin xyz="0 0 0" rpy="0 ${PI/2} 0"/>
+      <origin xyz="0 0 0" rpy="${PI/2} 0 0"/>
       <mass value="${wheelF_mass}"/>
       <cylinder_inertia  m="${wheelF_mass}" r="${wheelF_radius}" h="${wheelF_width}" />
@@ -29,12 +29,12 @@
   <!-- FL Wheel -->
   <joint name="wheelFL_joint" type="continuous">
-    <parent link="forklift_body"/>
+    <parent link="base_link"/>
     <child link="forklift_wheelFL"/>
-    <axis xyz="1 0 0"/>
-    <origin xyz="0.49389 -0.90059 0.34047"/>
+    <axis xyz="0 1 0"/>
+    <origin xyz="0 0.49389 0.34047"/> <!-- 0.49389 -0.90059 0.34047 -->
   </joint>
   <link name="forklift_wheelFL">
     <collision>
-      <origin xyz="0 0 0" rpy="0 ${PI/2} 0"/>
+      <origin xyz="0 0 0" rpy="${PI/2} 0 0"/>
       <geometry>
        <cylinder radius="${wheelF_radius}" length="${wheelF_width}" />
@@ -42,5 +42,5 @@
     </collision>
     <visual>
-      <origin xyz="0 0 0" rpy="0 0 0"/>
+      <origin xyz="0 0 0" rpy="0 0 ${PI/2}"/>
       <geometry>
        <mesh filename="package://forklift_description/meshes/forklift_wheel_front.dae"/>
@@ -48,5 +48,5 @@
     </visual>
     <inertial>
-      <origin xyz="0 0 0" rpy="0 ${PI/2} 0"/>
+      <origin xyz="0 0 0" rpy="${PI/2} 0 0"/>
       <mass value="${wheelF_mass}"/>
       <cylinder_inertia  m="${wheelF_mass}" r="${wheelF_radius}" h="${wheelF_width}" />

File: forklift_description/urdf/forklift_lift.xacro (robot description, xacro)
@@ -2,5 +2,5 @@
 <robot name="forklift" xmlns:xacro="http://www.ros.org/wiki/xacro">
   <joint name="lift1_joint" type="prismatic">
-    <parent link="forklift_body"/>
+    <parent link="base_link"/>
     <child link="forklift_lift1"/>
     <axis xyz="0 0 1"/>
@@ -9,23 +9,23 @@
   <link name="forklift_lift1">
     <collision>
-      <origin xyz="0 -1.44 0.695" rpy="0 0 0"/>
+      <origin xyz="0.55 0 0.695" rpy="0 0 0"/>
       <geometry>
-       <box size="1.2 0.1 1.25"/>
+       <box size="0.1 1.2 1.25"/>
       </geometry>
     </collision>
     <collision>
-      <origin xyz="0.32 -2.1 0.06" rpy="0 0 0"/>
+      <origin xyz="1.2 0.32 0.06" rpy="0 0 0"/>
       <geometry>
-       <box size="0.13 1.2 0.03"/>
+       <box size="1.2 0.13 0.03"/>
       </geometry>
     </collision>
     <collision>
-      <origin xyz="-0.32 -2.1 0.06" rpy="0 0 0"/>
+      <origin xyz="1.2 -0.32 0.06" rpy="0 0 0"/>
       <geometry>
-       <box size="0.13 1.2 0.03"/>
+       <box size="1.2 0.13 0.03"/>
       </geometry>
     </collision>
     <visual>
-      <origin xyz="0 0 0" rpy="0 0 0"/>
+      <origin xyz="-0.89856 0 0" rpy="0 0 ${PI/2}"/>
       <geometry>
        <mesh filename="package://forklift_description/meshes/forklift_lift1.dae"/>
@@ -33,11 +33,11 @@
     </visual>
     <inertial>
-      <origin xyz="0 -1.4 0.6" rpy="0 0 0"/>
+      <origin xyz="0.6 0 0.6" rpy="0 0 0"/>
       <mass value="${lift1_mass}"/>
-      <cube_inertia m="${lift1_mass}" w="1" h="1" d="0.3" />
+      <cube_inertia m="${lift1_mass}" w="0.3" h="1" d="1" />
     </inertial>
   </link>
   <joint name="lift2_joint" type="fixed">
-    <parent link="forklift_body"/>
+    <parent link="base_link"/>
     <child link="forklift_lift2"/>
     <axis xyz="0 0 1"/>
@@ -47,11 +47,11 @@
   <link name="forklift_lift2">
     <collision>
-      <origin xyz="0 -1.18 1.05" rpy="0 0 0"/>
+      <origin xyz="0.25 0 1.05" rpy="0 0 0"/>
       <geometry>
-       <box size="0.7 0.3 2"/>
+       <box size="0.3 0.7 2"/>
       </geometry>
     </collision>
     <visual>
-      <origin xyz="0 0 0" rpy="0 0 0"/>
+      <origin xyz="-0.89856 0 0" rpy="0 0 ${PI/2}"/>
       <geometry>
        <mesh filename="package://forklift_description/meshes/forklift_lift2.dae"/>
